Commit message: Add: Costmap Edit

File: src/simulation_launch/urdf/rover.urdf.xacro (robot description, xacro)
@@ -160,10 +160,10 @@
     <origin xyz="0.2 0 ${base_height/2 + 0.15}" rpy="0 0 0"/>
   </joint>
-  <!-- spoof zed camera tf tree-->
+  <!-- ✅ FIXED: ZED camera frame now attached to base_link (rotates with robot) -->
   <link name="zed_left_camera_frame"/>
   <joint name="zed_camera_joint" type="fixed">
-    <parent link="lidar_link"/>
+    <parent link="base_link"/>
     <child link="zed_left_camera_frame"/>
-    <origin xyz="0 0 0" rpy="0 0 0"/>
+    <origin xyz="0.2 0 ${base_height/2 + 0.15}" rpy="0 0 0"/>
   </joint>
   <!-- Gazebo 3D LiDAR Plugin (GPU accelerated) -->
@@ -191,4 +191,5 @@
           <min>0.3</min>
           <max>50.0</max>
+          <max>50.0</max>
           <resolution>0.01</resolution>
         </range>
